File: pcb/gator.sch (EAGLE design)
At the start: 2 parts, among them U1 ARDUINO_SHIELDLABEL, U2 WIFLY_GSX

Commit message: added some more libraries, refactored design to eliminate hdmi transmitter
Parts:
- removed U1: ARDUINO_SHIELDLABEL, SparkFun-Boards:ARDUINO_SHIELDLABEL
- added J1: MAGJACK-2, SparkFun-Connectors:MAGJACK-2
- added J2: POWER_JACKPTH, SparkFun-Connectors:POWER_JACKPTH
- added S1: (no value), SparkFun-Electromechanical:TAC_SWITCHPTH
- added SV1: (no value), con-ml:ML20
- added U$1: STM32F417, gator:STM32F417
- added U$2: XC3S250/500E-PQ208, SparkFun-DigitalIC:XC3S250/500E-PQ208
- added U$3: DP83848C, gator:DP83848C
- added X2: USB-A-S, SparkFun-Connectors:USB-A-S
- U2: value WIFLY_GSX -> USD-SOCKETNEW; device SparkFun:WIFLY_GSX -> SparkFun-Connectors:USD-SOCKETNEW
Changed lines of the file:
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@@
 </classes>
 <parts>
-<part name="U2" library="SparkFun" deviceset="WIFLY_GSX" device=""/>
-<part name="U1" library="SparkFun-Boards" deviceset="ARDUINO_SHIELD" device="LABEL"/>
+<part name="J1" library="SparkFun-Connectors" deviceset="MAGJACK-2" device=""/>
+<part name="U2" library="SparkFun-Connectors" deviceset="USD-SOCKET" device="NEW"/>
+<part name="X2" library="SparkFun-Connectors" deviceset="USB" device="-A-S"/>
+<part name="J2" library="SparkFun-Connectors" deviceset="POWER_JACK" device="PTH"/>
+<part name="S1" library="SparkFun-Electromechanical" deviceset="TAC_SWITCH" device="PTH"/>
+<part name="U$1" library="gator" deviceset="STM32F417" device=""/>
+<part name="U$2" library="SparkFun-DigitalIC" deviceset="XC3S250/500E-PQ208" device=""/>
+<part name="U$3" library="gator" deviceset="DP83848C" device=""/>
+<part name="SV1" library="con-ml" deviceset="ML20" device=""/>
 </parts>
 <sheets>
@@
 </plain>
 <instances>
-<instance part="U2" gate="G$1" x="-5.08" y="60.96" smashed="yes">
-<attribute name="NAME" x="-5.08" y="61.722" size="1.778" layer="95"/>
-<attribute name="VALUE" x="1.524" y="97.282" size="1.778" layer="96"/>
-</instance>
-<instance part="U1" gate="G$1" x="-71.12" y="68.58"/>
+<instance part="J1" gate="G$1" x="142.24" y="299.72"/>
+<instance part="U2" gate="G$1" x="172.72" y="259.08"/>
+<instance part="X2" gate="G$1" x="198.12" y="215.9"/>
+<instance part="J2" gate="G$1" x="200.66" y="279.4"/>
+<instance part="S1" gate="S" x="170.18" y="294.64"/>
+<instance part="U$1" gate="G$1" x="-233.68" y="269.24"/>
+<instance part="U$2" gate="G$1" x="-101.6" y="299.72"/>
+<instance part="U$3" gate="G$1" x="-83.82" y="129.54"/>
+<instance part="SV1" gate="1" x="2.54" y="144.78"/>
 </instances>
 <busses>

Commit message: Migrated to Spartan 6 and added more parts
Parts:
- removed SV1: (no value), con-ml:ML20
- removed U$2: XC3S250/500E-PQ208, SparkFun-DigitalIC:XC3S250/500E-PQ208
- removed U$3: DP83848C, gator:DP83848C
- removed U2: USD-SOCKETNEW, SparkFun-Connectors:USD-SOCKETNEW
- removed X2: USB-A-S, SparkFun-Connectors:USB-A-S
- added C1, C10, C12, C14, C15, C17, C18, C20, C3, C5, C8: 100n, SparkFun-Passives:CAP0603-CAP
- added C11, C2, C7: 470p, SparkFun-Passives:CAP0603-CAP
- added C13, C16, C19, C4, C6, C9: 2.2u, SparkFun-Passives:CAP0603-CAP
- added D1: REVPROT, SparkFun-DiscreteSemi:DIODEPTH
- added ETH_PHY: DP83848C, gator:DP83848C
- added FPGA: 6SLX9TQG144, xilinx_devices:6SLX9TQG144
- added HDMI: HDMI-TYPE-A-RECEPTICALFCI10029449, hdmi:HDMI-TYPE-A-RECEPTICALFCI10029449
- added JTAG: (no value), con-ml:ML20
- added MIC5219-3.3YM5_1, MIC5219-3.3YM5_2, MIC5219-5.0YM5: V_REG_LDOSMD, SparkFun-PowerIC:V_REG_LDOSMD
- added MICROSD: USD-SOCKETNEW, SparkFun-Connectors:USD-SOCKETNEW
- added NCP565ST12T3G, TLV1117-25CDCYR: (no value), microbuilder:LM1117SOT223-REFLOW
- added R1, R2, R3, R4, R7, R8: 10K, SparkFun-Passives:RESISTOR0603-RES
- added USBA: USB-A-S, SparkFun-Connectors:USB-A-S
- added WING: BOARDSIDE_16BIT_RIGHT, GadgetFactory_Pub:BOARDSIDE_16BIT_RIGHT
- U$1: value STM32F417 -> STM32F417VGT6; device gator:STM32F417 -> gator:STM32F417VGT6
- renumbered J1 to RJ45
Connections:
- new net +3V3: C8.1, C9.1, JTAG.1, MIC5219-3.3YM5_1.OUT, MICROSD.VCC, R4.2, WINGG$2.3V3, WINGG$3.3V3
- new net +5V: WINGG$2.5V, WINGG$3.5V
- new net /TRST: JTAG.3
- new net DBGACK: JTAG.19, R1.1
- new net DBGRQ: JTAG.17, R2.1
- new net GND: C1.1, C10.2, C11.2, C12.2, C13.2, C14.2, C15.2, C16.2, C17.2, C18.2, C19.2, C2.2, C20.2, C3.2, C4.2, C5.2, C6.2, C7.2, C8.2, C9.2, J2.GND, J2.GNDBREAK, JTAG.10, JTAG.12, JTAG.14, JTAG.16, JTAG.18, JTAG.20, JTAG.4, JTAG.6, JTAG.8, MIC5219-3.3YM5_1.GND, MIC5219-3.3YM5_2.GND, MIC5219-5.0YM5.GND, MICROSD.GND, MICROSD.SHIELD@1, MICROSD.SHIELD@3, NCP565ST12T3G.ADJ, R1.2, R2.2, R3.2, S1.1, S1.2, TLV1117-25CDCYR.ADJ, USBA.GND, WINGG$2.GND, WINGG$3.GND
- new net N$2: USBA.D-
- new net N$3: D1.A, J2.PWR
- new net N$4: C2.1, MIC5219-5.0YM5.BP
- new net N$5: MIC5219-3.3YM5_1.EN, R7.1
- new net N$6: C11.1, MIC5219-3.3YM5_2.BP
- new net N$7: C7.1, MIC5219-3.3YM5_1.BP
- new net N$8: MIC5219-3.3YM5_2.EN, R8.1
- new net NRST: C1.2, JTAG.15, R4.1, S1.3, S1.4
- new net RTCK: JTAG.11, R3.1
- new net SD_CLK: MICROSD.SCK
- new net SD_CMD: MICROSD.DI
- new net SD_D0: MICROSD.DO
- new net SD_D1: MICROSD.RSV
- new net SD_D2: MICROSD.NC
- new net SD_D3: MICROSD.CS
- new net TCLK/SWCLK: JTAG.9
- new net TDI: JTAG.5
- new net TDO/SWO: JTAG.13
- new net TMS/SWDIO: JTAG.7
- new net USB_DP: USBA.D+
- new net USB_EN: MIC5219-5.0YM5.EN
- new net USB_VBUS: C3.1, C4.1, MIC5219-5.0YM5.OUT, USBA.VBUS
- new net V+: C10.1, C14.1, C15.1, C18.1, C5.1, C6.1, D1.C, MIC5219-3.3YM5_1.IN, MIC5219-3.3YM5_2.IN, MIC5219-5.0YM5.IN, NCP565ST12T3G.IN, R7.2, R8.2, TLV1117-25CDCYR.IN
- new net VCC/2: C19.1, C20.1, TLV1117-25CDCYR.OUT, WINGG$2.2V5, WINGG$3.2V5
- new net VCCINT: C16.1, C17.1, NCP565ST12T3G.OUT
- new net VCCIO: C12.1, C13.1, MIC5219-3.3YM5_2.OUT
Other:
- moved on the sheet: J2, S1

Commit message: Finished arm cortex part
Connections:
- removed net USB_DP: USBA.D+
- new net N$1: U$1G$5.USB_FS_DP, USBA.D+
- new net TCK/SWCLK: U$1G$6.TCK/SWCLK
- net /TRST: now also U$1G$6.TRST
- net N$2: now also U$1G$5.USB_FS_DM
- net NRST: now also U$1G$6.NRST
- net SD_CLK: now also U$1G$4.SDIO_CLK
- net SD_CMD: now also U$1G$4.SDIO_CMD
- net SD_D0: now also U$1G$4.SDIO_D0
- net SD_D1: now also U$1G$4.SDIO_D1
- net SD_D2: now also U$1G$4.SDIO_D2
- net SD_D3: now also U$1G$4.SDIO_D3
- net TDI: now also U$1G$6.TDI
- net TDO/SWO: now also U$1G$6.TDO/SWO
- net TMS/SWDIO: now also U$1G$6.TMS/SWDIO
- net USB_EN: now also U$1G$5.USB_EN_ID
- net USB_VBUS: now also U$1G$5.USB_VBUS
Other:
- moved on the sheet: U$1G$2
Changed lines of the file:
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@@
 <instance part="P+11" gate="G$1" x="-53.34" y="429.26"/>
 <instance part="U$1" gate="G$1" x="-195.58" y="127"/>
-<instance part="U$1" gate="G$2" x="-142.24" y="106.68"/>
+<instance part="U$1" gate="G$2" x="-149.86" y="109.22"/>
+<instance part="U$1" gate="G$3" x="-104.14" y="129.54"/>
+<instance part="U$1" gate="G$4" x="-396.24" y="317.5"/>
+<instance part="U$1" gate="G$5" x="-238.76" y="396.24"/>
+<instance part="U$1" gate="G$6" x="-353.06" y="226.06"/>
+<instance part="U$1" gate="G$7" x="71.12" y="129.54"/>
+<instance part="U$1" gate="G$8" x="121.92" y="129.54"/>
+<instance part="U$1" gate="G$9" x="152.4" y="116.84"/>
 </instances>
 <busses>
@@
 <label x="-210.82" y="233.68" size="1.778" layer="95"/>
 </segment>
+<segment>
+<pinref part="U$1" gate="G$6" pin="TRST"/>
+<wire x1="-342.9" y1="231.14" x2="-340.36" y2="231.14" width="0.1524" layer="91"/>
+<label x="-340.36" y="231.14" size="1.778" layer="95"/>
+</segment>
 </net>
 <net name="TDI" class="0">
@@
 <label x="-210.82" y="266.7" size="1.778" layer="95"/>
 </segment>
+<segment>
+<pinref part="U$1" gate="G$6" pin="TDI"/>
+<wire x1="-342.9" y1="233.68" x2="-340.36" y2="233.68" width="0.1524" layer="91"/>
+<label x="-340.36" y="233.68" size="1.778" layer="95"/>
+</segment>
 </net>
 <net name="TMS/SWDIO" class="0">
@@
 <wire x1="-213.36" y1="279.4" x2="-210.82" y2="279.4" width="0.1524" layer="91"/>
 <label x="-210.82" y="279.4" size="1.778" layer="95"/>
+</segment>
+<segment>
+<pinref part="U$1" gate="G$6" pin="TMS/SWDIO"/>
+<wire x1="-342.9" y1="241.3" x2="-340.36" y2="241.3" width="0.1524" layer="91"/>
+<label x="-340.36" y="241.3" size="1.778" layer="95"/>
 </segment>
 </net>
@@
 <wire x1="-213.36" y1="236.22" x2="-210.82" y2="236.22" width="0.1524" layer="91"/>
 <label x="-210.82" y="236.22" size="1.778" layer="95"/>
+</segment>
+<segment>
+<pinref part="U$1" gate="G$6" pin="TDO/SWO"/>
+<wire x1="-342.9" y1="236.22" x2="-340.36" y2="236.22" width="0.1524" layer="91"/>
+<label x="-340.36" y="236.22" size="1.778" layer="95"/>
 </segment>
 </net>
@@
 <junction x="-284.48" y="299.72"/>
 <label x="-271.78" y="299.72" size="1.778" layer="95"/>
+</segment>
+<segment>
+<pinref part="U$1" gate="G$6" pin="NRST"/>
+<wire x1="-342.9" y1="228.6" x2="-340.36" y2="228.6" width="0.1524" layer="91"/>
+<label x="-340.36" y="228.6" size="1.778" layer="95"/>
 </segment>
 </net>
@@
 <label x="-355.6" y="317.5" size="1.778" layer="95"/>
 </segment>
+<segment>
+<pinref part="U$1" gate="G$4" pin="SDIO_D0"/>
+<wire x1="-386.08" y1="325.12" x2="-383.54" y2="325.12" width="0.1524" layer="91"/>
+<label x="-383.54" y="325.12" size="1.778" layer="95"/>
+</segment>
 </net>
 <net name="SD_D1" class="0">
@@
 <label x="-355.6" y="314.96" size="1.778" layer="95"/>
 </segment>
+<segment>
+<pinref part="U$1" gate="G$4" pin="SDIO_D1"/>
+<wire x1="-386.08" y1="327.66" x2="-383.54" y2="327.66" width="0.1524" layer="91"/>
+<label x="-383.54" y="327.66" size="1.778" layer="95"/>
+</segment>
 </net>
 <net name="SD_D2" class="0">
@@
 <label x="-355.6" y="332.74" size="1.778" layer="95"/>
 </segment>
+<segment>
+<pinref part="U$1" gate="G$4" pin="SDIO_D2"/>
+<wire x1="-386.08" y1="330.2" x2="-383.54" y2="330.2" width="0.1524" layer="91"/>
+<label x="-383.54" y="330.2" size="1.778" layer="95"/>
+</segment>
 </net>
 <net name="SD_D3" class="0">
@@
 <label x="-355.6" y="330.2" size="1.778" layer="95"/>
 </segment>
+<segment>
+<pinref part="U$1" gate="G$4" pin="SDIO_D3"/>
+<wire x1="-386.08" y1="332.74" x2="-383.54" y2="332.74" width="0.1524" layer="91"/>
+<label x="-383.54" y="332.74" size="1.778" layer="95"/>
+</segment>
 </net>
 <net name="SD_CLK" class="0">
@@
 <label x="-355.6" y="322.58" size="1.778" layer="95"/>
 </segment>
+<segment>
+<pinref part="U$1" gate="G$4" pin="SDIO_CLK"/>
+<wire x1="-386.08" y1="322.58" x2="-383.54" y2="322.58" width="0.1524" layer="91"/>
+<label x="-383.54" y="322.58" size="1.778" layer="95"/>
+</segment>
 </net>
 <net name="SD_CMD" class="0">
@@
 <label x="-355.6" y="327.66" size="1.778" layer="95"/>
 </segment>
+<segment>
+<pinref part="U$1" gate="G$4" pin="SDIO_CMD"/>
+<wire x1="-386.08" y1="320.04" x2="-383.54" y2="320.04" width="0.1524" layer="91"/>
+<label x="-383.54" y="320.04" size="1.778" layer="95"/>
+</segment>
 </net>
 <net name="USB_DM" class="0">
@@
 <label x="-210.82" y="284.48" size="1.778" layer="95"/>
 </segment>
-<segment>
-<wire x1="-233.68" y1="403.86" x2="-238.76" y2="403.86" width="0.1524" layer="91"/>
-<label x="-246.38" y="403.86" size="1.778" layer="95"/>
-</segment>
 </net>
 <net name="USB_DP" class="0">
@@
 <wire x1="-213.36" y1="281.94" x2="-210.82" y2="281.94" width="0.1524" layer="91"/>
 <label x="-210.82" y="281.94" size="1.778" layer="95"/>
-</segment>
-<segment>
-<label x="-246.38" y="408.94" size="1.778" layer="95"/>
-<wire x1="-215.9" y1="408.94" x2="-215.9" y2="401.32" width="0.1524" layer="91"/>
-<pinref part="USBA" gate="G$1" pin="D+"/>
-<wire x1="-215.9" y1="401.32" x2="-213.36" y2="401.32" width="0.1524" layer="91"/>
-<wire x1="-238.76" y1="408.94" x2="-215.9" y2="408.94" width="0.1524" layer="91"/>
 </segment>
 </net>
@@
 <wire x1="-248.92" y1="391.16" x2="-233.68" y2="391.16" width="0.1524" layer="91"/>
 <wire x1="-233.68" y1="391.16" x2="-223.52" y2="391.16" width="0.1524" layer="91"/>
-<wire x1="-223.52" y1="391.16" x2="-223.52" y2="396.24" width="0.1524" layer="91"/>
-<pinref part="USBA" gate="G$1" pin="VBUS"/>
-<wire x1="-223.52" y1="396.24" x2="-213.36" y2="396.24" width="0.1524" layer="91"/>
 <pinref part="C3" gate="G$1" pin="1"/>
 <wire x1="-233.68" y1="388.62" x2="-233.68" y2="391.16" width="0.1524" layer="91"/>
@@
 <wire x1="-223.52" y1="388.62" x2="-223.52" y2="391.16" width="0.1524" layer="91"/>
 <junction x="-233.68" y="391.16"/>
+<label x="-248.92" y="391.16" size="1.778" layer="95"/>
+<pinref part="USBA" gate="G$1" pin="VBUS"/>
+<wire x1="-218.44" y1="396.24" x2="-213.36" y2="396.24" width="0.1524" layer="91"/>
+<pinref part="U$1" gate="G$5" pin="USB_VBUS"/>
+<wire x1="-228.6" y1="408.94" x2="-218.44" y2="408.94" width="0.1524" layer="91"/>
+<wire x1="-218.44" y1="408.94" x2="-218.44" y2="396.24" width="0.1524" layer="91"/>
+<wire x1="-223.52" y1="391.16" x2="-218.44" y2="391.16" width="0.1524" layer="91"/>
+<wire x1="-218.44" y1="391.16" x2="-218.44" y2="396.24" width="0.1524" layer="91"/>
 <junction x="-223.52" y="391.16"/>
-<label x="-248.92" y="391.16" size="1.778" layer="95"/>
-</segment>
-</net>
-<net name="N$2" class="0">
-<segment>
-<pinref part="USBA" gate="G$1" pin="D-"/>
-<wire x1="-213.36" y1="398.78" x2="-218.44" y2="398.78" width="0.1524" layer="91"/>
-<wire x1="-218.44" y1="398.78" x2="-218.44" y2="403.86" width="0.1524" layer="91"/>
-<wire x1="-218.44" y1="403.86" x2="-233.68" y2="403.86" width="0.1524" layer="91"/>
+<junction x="-218.44" y="396.24"/>
 </segment>
 </net>
@@
 <label x="-210.82" y="287.02" size="1.778" layer="95"/>
 </segment>
+<segment>
+<pinref part="U$1" gate="G$5" pin="USB_EN_ID"/>
+<wire x1="-228.6" y1="406.4" x2="-226.06" y2="406.4" width="0.1524" layer="91"/>
+<label x="-231.14" y="403.86" size="1.778" layer="95"/>
+</segment>
 </net>
 <net name="+5V" class="0">
@@
 </segment>
 </net>
+<net name="N$1" class="0">
+<segment>
+<pinref part="U$1" gate="G$5" pin="USB_FS_DP"/>
+<pinref part="USBA" gate="G$1" pin="D+"/>
+<wire x1="-228.6" y1="401.32" x2="-213.36" y2="401.32" width="0.1524" layer="91"/>
+</segment>
+</net>
+<net name="N$2" class="0">
+<segment>
+<pinref part="USBA" gate="G$1" pin="D-"/>
+<pinref part="U$1" gate="G$5" pin="USB_FS_DM"/>
+<wire x1="-213.36" y1="398.78" x2="-228.6" y2="398.78" width="0.1524" layer="91"/>
+</segment>
+</net>
+<net name="TCK/SWCLK" class="0">
+<segment>
+<pinref part="U$1" gate="G$6" pin="TCK/SWCLK"/>
+<wire x1="-342.9" y1="238.76" x2="-340.36" y2="238.76" width="0.1524" layer="91"/>
+<label x="-340.36" y="238.76" size="1.778" layer="95"/>
+</segment>
+</net>

Commit message: Assigned many of the FPGA pins, cleaned up HDMI connector
Parts:
- removed HDMI: HDMI-TYPE-A-RECEPTICALFCI10029449, hdmi:HDMI-TYPE-A-RECEPTICALFCI10029449
- added C21: 10u, SparkFun-Passives:CAP0603-CAP
- added C22, C23, C24, C25, C26, C27, C29, C31: 100n, SparkFun-Passives:CAP0603-CAP
- added C28: 470p, SparkFun-Passives:CAP0603-CAP
- added C30: 2.2u, SparkFun-Passives:CAP0603-CAP
- added MIC5219-5.0YM1: V_REG_LDOSMD, SparkFun-PowerIC:V_REG_LDOSMD
- added R10, R5, R6, R9: 51, SparkFun-Passives:RESISTOR0603-RES
- added R11, R12, R13, R17, R18: 2K2, SparkFun-Passives:RESISTOR0603-RES
- added R14, R15: 110, SparkFun-Passives:RESISTOR0603-RES
- added R16: 4K87, SparkFun-Passives:RESISTOR0603-RES
- added R19: 5K6, SparkFun-Passives:RESISTOR0603-RES
- added R20: 10K, SparkFun-Passives:RESISTOR0603-RES
- added U$2: HDMI_A, gator:HDMI_A
Connections:
- new net 50MHZ_OSC: ETH_PHY.X1, U$1G$3.RMII_REF_CLK
- new net A16: U$1G$2.A16
- new net A17: U$1G$2.A17
- new net A18: U$1G$2.A18
- new net A19: U$1G$2.A19
- new net A20: U$1G$2.A20
- new net A21: U$1G$2.A21
- new net A22: U$1G$2.A22
- new net A23: U$1G$2.A23
- new net CEC: FPGAB0.IO_L65N_SCP2_0, U$2.CEC
- new net CSO_B: FPGAB2.IO_L65N_CSO_B_2
- new net D0: FPGAB2.IO_L03P_D0_DIN_MISO_MISO1_2, U$1G$2.A0/D0
- new net D1: FPGAB2.IO_L12P_D1_MISO2_2, U$1G$2.A1/D1
- new net D10: FPGAB2.IO_L13N_D10_2, U$1G$2.A10/D10
- new net D11: FPGAB2.IO_L14P_D11_2, U$1G$2.A11/D11
- new net D12: FPGAB2.IO_L14N_D12_2, U$1G$2.A12/D12
- new net D13: FPGAB2.IO_L30P_GCLK1_D13_2, U$1G$2.A13/D13
- new net D14: FPGAB2.IO_L31P_GCLK31_D14_2, U$1G$2.A14/D14
- new net D15: FPGAB2.IO_L31N_GCLK30_D15_2, U$1G$2.A15/D15
- new net D2: FPGAB2.IO_L12N_D2_MISO3_2, U$1G$2.A2/D2
- new net D3: FPGAB2.IO_L49P_D3_2, U$1G$2.A3/D3
- new net D4: FPGAB2.IO_L49N_D4_2, U$1G$2.A4/D4
- new net D5: FPGAB2.IO_L62P_D5_2, U$1G$2.A5/D5
- new net D6: FPGAB2.IO_L62N_D6_2, U$1G$2.A6/D6
- new net D7: FPGAB2.IO_L48P_D7_2, U$1G$2.A7/D7
- new net D8: FPGAB2.IO_L64P_D8_2, U$1G$2.A8/D8
- new net D9: FPGAB2.IO_L64N_D9_2, U$1G$2.A9/D9
- new net DDC_CLK: FPGAB0.IO_L65P_SCP3_0
- new net DDC_DATA: FPGAB0.IO_L66N_SCP0_0
- new net DONE: FPGAB2.DONE_2
- new net FSMC_CLK: U$1G$2.CLK
- new net HDMI_5V: C29.1, C30.1, MIC5219-5.0YM1.OUT, U$2.+5V
- new net HDMI_DETECT: FPGAB0.IO_L66P_SCP1_0, R19.1, R20.2
- new net INIT_B: FPGAB2.IO_L65P_INIT_B_2, U$1G$9.PB0
- new net LED_ACT: ETH_PHY.LED_ACT/COL/AN_EN, R13.1, RJ45.YLED-
- new net LED_LINK: ETH_PHY.LED_LINK/AN0, R11.1, RJ45.GLED-
- new net MII_INT: ETH_PHY.PWR_DOWN/INT, U$1G$3.MII_INT
- new net MII_MDC: ETH_PHY.MDC, U$1G$3.MII_MDC
- new net MII_MDIO: ETH_PHY.MDIO, U$1G$3.MII_MDIO
- new net MII_RXD0: ETH_PHY.RXD_0/PHYAD1, U$1G$3.MII_RXD0
- new net MII_RXD1: ETH_PHY.RXD_1/PHYAD1, U$1G$3.MII_RXD1
- new net MII_RX_ER: ETH_PHY.RX_ER/MDIX_EN, U$1G$3.MII_RX_ER
- new net MII_TXD0: ETH_PHY.TXD_0, U$1G$3.MII_TXD0
- new net MII_TXD1: ETH_PHY.TXD_1, U$1G$3.MII_TXD1
- new net MII_TX_EN: ETH_PHY.TX_EN, U$1G$3.MII_TX_EN
- new net N$10: ETH_PHY.RD-, R9.1, RJ45.RD-
- new net N$11: ETH_PHY.TD+, R6.1, RJ45.TD+
- new net N$12: ETH_PHY.TD-, R5.1, RJ45.TD-
- new net N$13: R14.1, RJ45.YLED+
- new net N$14: R15.2, RJ45.GLED+
- new net N$15: C28.1, MIC5219-5.0YM1.BP
- new net N$16: ETH_PHY.RBIAS, R16.2
- new net N$17: ETH_PHY.LED_SPEED/AN1, R12.1
- new net N$18: ETH_PHY.TXD_3, R18.2
- new net N$22: R19.2, U$2.DETECT
- new net N$9: ETH_PHY.RD+, R10.1, RJ45.RD+
- new net NBL0: U$1G$2.NBL0
- new net NBL1: U$1G$2.NBL1
- new net NE1: U$1G$2.NE1
- new net NL: U$1G$2.NL
- new net NOE: U$1G$2.NOE
- new net NWAIT: U$1G$2.NWAIT
- new net NWE: U$1G$2.NWE
- new net PFB: C21.1, C22.1, C23.1, ETH_PHY.PFBIN1, ETH_PHY.PFBIN2, ETH_PHY.PFBOUT
- new net PROGRAM_B: FPGAB2.PROGRAM_B_2, U$1G$9.PB1
- new net RMII_CRSDV: ETH_PHY.RX_DV/MII_MODE, R17.1, U$1G$3.RMII_CRSDV
- new net RMII_REF_CLK: ETH_PHY.25MHZ_OUT
- new net TMDS_CLKN: FPGAB0.IO_L64N_SCP4_0, U$2.TMDS_CLKN
- new net TMDS_CLKP: FPGAB0.IO_L64P_SCP5_0, U$2.TMDS_CLKP
- new net TMDS_D0N: FPGAB0.IO_L63N_SCP6_0, U$2.TMDS_D0N
- new net TMDS_D0P: FPGAB0.IO_L63P_SCP7_0, U$2.TMDS_D0P
- new net TMDS_D1N: FPGAB0.IO_L62N_VREF_0, U$2.TMDS_D1N
- new net TMDS_D1P: FPGAB0.IO_L62P_0, U$2.TMDS_D1P
- new net TMDS_D2N: FPGAB0.IO_L37N_GCLK12_0, U$2.TMDS_D2N
- new net TMDS_D2P: FPGAB0.IO_L37P_GCLK13_0, U$2.TMDS_D2P
- new net WING_A1: FPGAB1.IO_L47N_1, WINGG$1.A1
- new net WING_A10: FPGAB1.IO_L42P_GCLK7_1, WINGG$1.A10
- new net WING_A11: FPGAB1.IO_L41N_GCLK8_1, WINGG$1.A11
- new net WING_A12: FPGAB1.IO_L41P_GCLK9_IRDY1_1, WINGG$1.A12
- new net WING_A13: FPGAB1.IO_L40N_GCLK10_1, WINGG$1.A13
- new net WING_A14: FPGAB1.IO_L40P_GCLK11_1, WINGG$1.A14
- new net WING_A15: FPGAB1.IO_L34N_1, WINGG$1.A15
- new net WING_A16: FPGAB1.IO_L34P_1, WINGG$1.A16
- new net WING_A2: FPGAB1.IO_L47P_1, WINGG$1.A2
- new net WING_A3: FPGAB1.IO_L46N_1, WINGG$1.A3
- new net WING_A4: FPGAB1.IO_L46P_1, WINGG$1.A4
- new net WING_A5: FPGAB1.IO_L45N_1, WINGG$1.A5
- new net WING_A6: FPGAB1.IO_L45P_1, WINGG$1.A6
- new net WING_A7: FPGAB1.IO_L43N_GCLK4_1, WINGG$1.A7
- new net WING_A8: FPGAB1.IO_L43P_GCLK5_1, WINGG$1.A8
- new net WING_A9: FPGAB1.IO_L42N_GCLK6_TRDY1_1, WINGG$1.A9
- net +3V3: now also C24.1, C25.1, C26.1, C27.1, ETH_PHY.AVDD33, ETH_PHY.IOVDD33(1), ETH_PHY.IOVDD33(2), FPGAB0.VCCO_0@000, FPGAB0.VCCO_0@001, FPGAB0.VCCO_0@002, FPGAB1.VCCO_1@000, FPGAB1.VCCO_1@001, FPGAB1.VCCO_1@002, FPGAB2.VCCO_2@000, FPGAB2.VCCO_2@001, FPGAB3.VCCO_3@000, FPGAB3.VCCO_3@001, FPGAB3.VCCO_3@002, FPGABVCCAUX.VCCAUX@000, FPGABVCCAUX.VCCAUX@001, FPGABVCCAUX.VCCAUX@002, FPGABVCCAUX.VCCAUX@003, FPGABVCCAUX.VCCAUX@004, R10.2, R11.2, R12.2, R13.2, R14.2, R15.1, R17.2, R5.2, R6.2, R9.2, RJ45.RCT, RJ45.TCT
- net GND: now also C21.2, C22.2, C23.2, C24.2, C25.2, C26.2, C27.2, C28.2, C29.2, C30.2, C31.2, ETH_PHY.AGND1, ETH_PHY.AGND2, ETH_PHY.DGND, ETH_PHY.IOGND, ETH_PHY.IOGND2, FPGABGND.GND@000, FPGABGND.GND@001, FPGABGND.GND@002, FPGABGND.GND@003, FPGABGND.GND@004, FPGABGND.GND@005, FPGABGND.GND@006, FPGABGND.GND@007, FPGABGND.GND@008, FPGABGND.GND@009, FPGABGND.GND@010, FPGABGND.GND@011, FPGABGND.GND@012, MIC5219-5.0YM1.GND, R16.1, R18.1, R20.1, RJ45.SHIELD, U$2.GND, U$2.TMDS_CLK_SHLD, U$2.TMDS_D0_SHLD, U$2.TMDS_D1_SHLD, U$2.TMDS_D2_SHLD
- net NRST: now also ETH_PHY.RESET_N
- net USB_EN: now also MIC5219-5.0YM1.EN
- net V+: now also C31.1, MIC5219-5.0YM1.IN
- net VCCINT: now also FPGABVCCINT.VCCINT@000, FPGABVCCINT.VCCINT@001, FPGABVCCINT.VCCINT@002, FPGABVCCINT.VCCINT@003, FPGABVCCINT.VCCINT@004
Other:
- moved on the sheet: C1, ETH_PHY, FPGAB0, R4, RJ45, S1, U$1G$1, U$1G$2, U$1G$7, U$1G$8, WINGG$1
